Commit message: fix: match original opencat-gym to achieve walking (10 bugs fixed)
Critical fixes that enabled successful locomotion training:

1. Joint mapping: [0,4,1,5,2,6,3,7] pointed 3 actions at FIXED joints
   (battery, paw_front_left/right), leaving rear legs uncontrolled.
   Now uses dynamic discovery → [1,2,4,5,7,8,10,11].

2. Stability penalty: raw angular velocity squared (100x too large).
   Now applies ×0.1 scaling + clip(-1,1) before squaring.

3. Arm contact: break after first contact → max +1/step.
   Now checks each link independently → max +4/step.

4. Reset method: fast reset (resetBasePosition) could leave residual
   physics state. Now uses resetSimulation() matching original.

5. Initial pose: all joints at 50° vs original [50,0,50,0,50,0,50,0]°
   (shoulders/hips angled, elbows/knees straight).

6. URDF joint limits: effort=0.2, velocity=31.4 vs original effort=0,
   velocity=0 + changeDynamics. Now matches original.

7. Joint angles: tracked in Python (open-loop) vs read from PyBullet
   (closed-loop feedback). Now reads actual physics state each step.

8. stepSimulation timing: 3 steps concentrated after motor command vs
   original's distributed timing. Now matches original's 3-step pattern.

9. start_pos: [0,0,0.1] → [0,0,0.08] matching original.

10. joint_history init: zeros → filled with initial pose.

Also: simplified curriculum to single 2M-step stage, added A/B test
and log comparison scripts.

Result: reward 1180 at 2M steps (matches baseline 1120), robot walks
with 0% arm contact, 0.077m avg height, 3.9° avg tilt.

Co-Authored-By: Claude Opus 4.6 (1M context) <noreply@anthropic.com>

File: jprobot/models/bittle_esp32.urdf (robot description, URDF)
Before this commit: robot BittleX, 14 links, 13 joints
Joints:
- joint elbow_left: limit lower=-1.57 upper=1.57 effort=0.2 velocity=31.4 -> lower=-1.57 upper=1.57 effort=0 velocity=0
- joint elbow_right: limit lower=-1.57 upper=1.57 effort=0.2 velocity=31.4 -> lower=-1.57 upper=1.57 effort=0 velocity=0
- joint hip_left: limit lower=-1.57 upper=2.0 effort=0.2 velocity=31.4 -> lower=-1.57 upper=2.00 effort=0 velocity=0
- joint hip_right: limit lower=-1.57 upper=2.0 effort=0.2 velocity=31.4 -> lower=-1.57 upper=2.00 effort=0 velocity=0
- joint knee_left: limit lower=-1.57 upper=1.57 effort=0.2 velocity=31.4 -> lower=-1.57 upper=1.57 effort=0 velocity=0
- joint knee_right: limit lower=-1.57 upper=1.57 effort=0.2 velocity=31.4 -> lower=-1.57 upper=1.57 effort=0 velocity=0
- joint shoulder_left: limit lower=-1.57 upper=1.57 effort=0.2 velocity=31.4 -> lower=-1.57 upper=1.57 effort=0 velocity=0
- joint shoulder_right: limit lower=-1.57 upper=1.57 effort=0.2 velocity=31.4 -> lower=-1.57 upper=1.57 effort=0 velocity=0
